File: mcp2562.kicad_sch (KiCad schematic)
At the start: 5 parts, among them Q701 BSS84, U701 MCP2558FD-xSN

Commit message: jk im stupid forgot to route the flash
Parts:
- renumbered C701 to C1001, C702 to C1002, Q701 to Q1001, R701 to R1001, U701 to U1001
Changed lines of the file:
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@@
 		(dnp no)
 		(fields_autoplaced yes)
-		(property "Reference" "U701"
+		(property "Reference" "U?"
 			(at 130.4133 72.39 0)
 			(effects
@@
 					(unit 1)
 				)
-				(path "/0aeff2df-21bc-4c76-95d6-83ff8577a8db/479988e2-73e3-4e6d-8b3c-5b8d2874850c/a5605b2d-f7ac-45f3-aba3-2f27c488895b/36677952-db68-4370-87fc-67a2e82899d4"
-					(reference "U701")
+				(path "/0aeff2df-21bc-4c76-95d6-83ff8577a8db/479988e2-73e3-4e6d-8b3c-5b8d2874850c/c9adf87a-8f92-44b6-917f-4b9ab2f21739"
+					(reference "U?")
 					(unit 1)
 				)
@@
 		(dnp no)
 		(fields_autoplaced yes)
-		(property "Reference" "Q701"
+		(property "Reference" "Q?"
 			(at 200.66 73.6599 0)
 			(effects
@@
 					(unit 1)
 				)
-				(path "/0aeff2df-21bc-4c76-95d6-83ff8577a8db/479988e2-73e3-4e6d-8b3c-5b8d2874850c/a5605b2d-f7ac-45f3-aba3-2f27c488895b/36677952-db68-4370-87fc-67a2e82899d4"
-					(reference "Q701")
+				(path "/0aeff2df-21bc-4c76-95d6-83ff8577a8db/479988e2-73e3-4e6d-8b3c-5b8d2874850c/c9adf87a-8f92-44b6-917f-4b9ab2f21739"
+					(reference "Q?")
 					(unit 1)
 				)
@@
 					(unit 1)
 				)
-				(path "/0aeff2df-21bc-4c76-95d6-83ff8577a8db/479988e2-73e3-4e6d-8b3c-5b8d2874850c/a5605b2d-f7ac-45f3-aba3-2f27c488895b/36677952-db68-4370-87fc-67a2e82899d4"
+				(path "/0aeff2df-21bc-4c76-95d6-83ff8577a8db/479988e2-73e3-4e6d-8b3c-5b8d2874850c/c9adf87a-8f92-44b6-917f-4b9ab2f21739"
 					(reference "#PWR0703")
 					(unit 1)
@@
 		(on_board yes)
 		(dnp no)
-		(property "Reference" "C701"
+		(property "Reference" "C?"
 			(at 108.458 64.262 0)
 			(effects
@@
 					(unit 1)
 				)
-				(path "/0aeff2df-21bc-4c76-95d6-83ff8577a8db/479988e2-73e3-4e6d-8b3c-5b8d2874850c/a5605b2d-f7ac-45f3-aba3-2f27c488895b/36677952-db68-4370-87fc-67a2e82899d4"
-					(reference "C701")
+				(path "/0aeff2df-21bc-4c76-95d6-83ff8577a8db/479988e2-73e3-4e6d-8b3c-5b8d2874850c/c9adf87a-8f92-44b6-917f-4b9ab2f21739"
+					(reference "C?")
 					(unit 1)
 				)
@@
 					(unit 1)
 				)
-				(path "/0aeff2df-21bc-4c76-95d6-83ff8577a8db/479988e2-73e3-4e6d-8b3c-5b8d2874850c/a5605b2d-f7ac-45f3-aba3-2f27c488895b/36677952-db68-4370-87fc-67a2e82899d4"
+				(path "/0aeff2df-21bc-4c76-95d6-83ff8577a8db/479988e2-73e3-4e6d-8b3c-5b8d2874850c/c9adf87a-8f92-44b6-917f-4b9ab2f21739"
 					(reference "#PWR0701")
 					(unit 1)
@@
 		(on_board yes)
 		(dnp no)
-		(property "Reference" "C702"
+		(property "Reference" "C?"
 			(at 107.442 93.726 0)
 			(effects
@@
 					(unit 1)
 				)
-				(path "/0aeff2df-21bc-4c76-95d6-83ff8577a8db/479988e2-73e3-4e6d-8b3c-5b8d2874850c/a5605b2d-f7ac-45f3-aba3-2f27c488895b/36677952-db68-4370-87fc-67a2e82899d4"
-					(reference "C702")
+				(path "/0aeff2df-21bc-4c76-95d6-83ff8577a8db/479988e2-73e3-4e6d-8b3c-5b8d2874850c/c9adf87a-8f92-44b6-917f-4b9ab2f21739"
+					(reference "C?")
 					(unit 1)
 				)
@@
 					(unit 1)
 				)
-				(path "/0aeff2df-21bc-4c76-95d6-83ff8577a8db/479988e2-73e3-4e6d-8b3c-5b8d2874850c/a5605b2d-f7ac-45f3-aba3-2f27c488895b/36677952-db68-4370-87fc-67a2e82899d4"
+				(path "/0aeff2df-21bc-4c76-95d6-83ff8577a8db/479988e2-73e3-4e6d-8b3c-5b8d2874850c/c9adf87a-8f92-44b6-917f-4b9ab2f21739"
 					(reference "#PWR0702")
 					(unit 1)
@@
 		(dnp no)
 		(fields_autoplaced yes)
-		(property "Reference" "R701"
+		(property "Reference" "R?"
 			(at 199.39 83.8199 90)
 			(effects
@@
 					(unit 1)
 				)
-				(path "/0aeff2df-21bc-4c76-95d6-83ff8577a8db/479988e2-73e3-4e6d-8b3c-5b8d2874850c/a5605b2d-f7ac-45f3-aba3-2f27c488895b/36677952-db68-4370-87fc-67a2e82899d4"
-					(reference "R701")
-					(unit 1)
-				)
+				(path "/0aeff2df-21bc-4c76-95d6-83ff8577a8db/479988e2-73e3-4e6d-8b3c-5b8d2874850c/c9adf87a-8f92-44b6-917f-4b9ab2f21739"
+					(reference "R?")
+					(unit 1)
+				)

Commit message: fixed like a bunch of things, power and new xcvr and lights and other goodies, also started layout
Parts:
- removed C1002: 100n, Capacitor_SMD:C_0603_1608Metric_Pad1.08x0.95mm_HandSolder, symbol bfr_capacitors:06035C104KAT2A
- removed U1001: MCP2558FD-xSN, Package_SO:SOIC-8_3.9x4.9mm_P1.27mm, symbol Interface_CAN_LIN:MCP2558FD-xSN
- added D701, D702: White, Diode_SMD:D_0603_1608Metric_Pad1.05x0.95mm_HandSolder, symbol bfr_diodes:KT-0603W
- added JP701: CAN_TERM, Jumper:SolderJumper-2_P1.3mm_Open_RoundedPad1.0x1.5mm, symbol Jumper:SolderJumper_2_Open
- added Q702: BSS84, Package_TO_SOT_SMD:SOT-23, symbol Transistor_FET:BSS84
- added R701: 120, Resistor_SMD:R_0402_1005Metric_Pad0.72x0.64mm_HandSolder, symbol bfr_resistors:RMCF0402FT120R
- added R703: 120, Resistor_SMD:R_0603_1608Metric_Pad0.98x0.95mm_HandSolder, symbol bfr_resistors:RMCF0603FT120R
- added U701: TCAN334G, Package_TO_SOT_SMD:TSOT-23-8, symbol Interface_CAN_LIN:TCAN334G
- renumbered C1001 to C701, Q1001 to Q701, R1001 to R702
Connections:
- net 5V is gone; now on net 3V3: C701.1
- net 3V3: now also Q701.2 (S), Q702.2 (S), U701.3 (VCC); no longer Q701.3 (D)
- net CANH: now also JP701.1 (A), U701.7 (CANH)
- net CANL: now also R701.1, U701.6 (CANL)
- net CRX: now also Q702.1 (G), U701.4 (RXD)
- net CTX: now also U701.1 (TXD)
- net GND: now also D701.1 (K), D702.1 (K), U701.2 (GND), U701.5 (SHDN), U701.8 (STB); no longer R702.1
- net at R702.2: now also Q701.3 (D); no longer Q701.2 (S)
- new net: JP701.2 (B), R701.2
- new net: D701.2 (A), R702.1
- new net: D702.2 (A), R703.1
- new net: Q702.3 (D), R703.2
Other:
- note added: "RX LED"
- note added: "TX LED"
- note removed: "Debug LED"
- moved on the sheet: Q701, R702
