File: nor_flash.kicad_sch (KiCad schematic)
At the start: 11 parts, among them U901 MX25R3235FM2xx1

Commit message: jk im stupid forgot to route the flash
Parts:
- U901: Created By (none) -> Manual Entry; Digikey P/N (none) -> MX25R3235FM2IL0-ND; JLC Basic Part (none) -> No; LCSC P/N (none) -> C2802828; Manufacturer (none) -> Macronix; Manufacturer P/N (none) -> MX25R3235FM2IL0; Mouser P/N (none) -> 95-25R3235FM2IL0TR; Order From (none) -> Digikey
Changed lines of the file:
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@@
+			)
+		)
+		(property "Manufacturer P/N" "MX25R3235FM2IL0"
+			(at 113.03 71.12 0)
+			(effects
+				(font
+					(size 1.27 1.27)
+				)
+				(hide yes)
+			)
+		)
+		(property "Manufacturer" "Macronix"
+			(at 113.03 71.12 0)
+			(effects
+				(font
+					(size 1.27 1.27)
+				)
+				(hide yes)
+			)
+		)
+		(property "Digikey P/N" "MX25R3235FM2IL0-ND"
+			(at 113.03 71.12 0)
+			(effects
+				(font
+					(size 1.27 1.27)
+				)
+				(hide yes)
+			)
+		)
+		(property "Mouser P/N" "95-25R3235FM2IL0TR "
+			(at 113.03 71.12 0)
+			(effects
+				(font
+					(size 1.27 1.27)
+				)
+				(hide yes)
+			)
+		)
+		(property "LCSC P/N" "C2802828"
+			(at 113.03 71.12 0)
+			(effects
+				(font
+					(size 1.27 1.27)
+				)
+				(hide yes)
+			)
+		)
+		(property "JLC Basic Part" "No"
+			(at 113.03 71.12 0)
+			(effects
+				(font
+					(size 1.27 1.27)
+				)
+				(hide yes)
+			)
+		)
+		(property "Order From" "Digikey"
+			(at 113.03 71.12 0)
+			(effects
+				(font
+					(size 1.27 1.27)
+				)
+				(hide yes)
+			)
+		)
+		(property "Created By" "Manual Entry"
+			(at 113.03 71.12 0)
+			(effects
+				(font
+					(size 1.27 1.27)
+				)
+				(hide yes)
+			)
+		)
+		(property "Pretty Name" ""
+			(at 113.03 71.12 0)
+			(effects
+				(font
+					(size 1.27 1.27)
+				)
+				(hide yes)
 			)
 		)

Commit message: fixed like a bunch of things, power and new xcvr and lights and other goodies, also started layout
Parts:
- removed C902: 1u, Capacitor_SMD:C_0402_1005Metric_Pad0.74x0.62mm_HandSolder, symbol bfr_capacitors:CL05A105KA5NQNC
- removed C903: 10u, Capacitor_SMD:C_0603_1608Metric_Pad1.08x0.95mm_HandSolder, symbol bfr_capacitors:CL10A106MA8NRNC
- added C902, C903: 100n, Capacitor_SMD:C_0402_1005Metric_Pad0.74x0.62mm_HandSolder, symbol bfr_capacitors:CL05B104KB54PNC
- renumbered D905 to D901, R903 to R901, R904 to R902, R905 to R903, R906 to R904, R907 to R905, R908 to R906
Connections:
- net 3V3: now also C902.1, C903.1
- net GND: now also C902.2, C903.2
Other:
- moved on the sheet: C901, D901, R901, R902, R903, R904, R905, R906, U901
