File: stm32f103_decoupling.kicad_sch (KiCad schematic)
At the start: 4 parts

Commit message: fixed like a bunch of things, power and new xcvr and lights and other goodies, also started layout
Parts:
- added C1601: 100n, Capacitor_SMD:C_0402_1005Metric_Pad0.74x0.62mm_HandSolder, symbol bfr_capacitors:CL05B104KB54PNC
- C1602: renamed from C1101; footprint Capacitor_SMD:C_0603_1608Metric_Pad1.08x0.95mm_HandSolder -> Capacitor_SMD:C_0402_1005Metric_Pad0.74x0.62mm_HandSolder; symbol bfr_capacitors:06035C104KAT2A -> bfr_capacitors:CL05B104KB54PNC; Created by capacitor_generator.py script using capacitor_bible_spec.txt -> capacitor_generator.py script using jlcbasic_additional_cap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; LCSC P/N C14663 -> C307331; Pretty Name 100nF 16V 0603 Capacitor -> 100nF X7R 50V 0402 Capacitor
- C1603: renamed from C1102; footprint Capacitor_SMD:C_0603_1608Metric_Pad1.08x0.95mm_HandSolder -> Capacitor_SMD:C_0402_1005Metric_Pad0.74x0.62mm_HandSolder; symbol bfr_capacitors:06035C104KAT2A -> bfr_capacitors:CL05B104KB54PNC; Created by capacitor_generator.py script using capacitor_bible_spec.txt -> capacitor_generator.py script using jlcbasic_additional_cap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; LCSC P/N C14663 -> C307331; Pretty Name 100nF 16V 0603 Capacitor -> 100nF X7R 50V 0402 Capacitor
- C1604: renamed from C1103; footprint Capacitor_SMD:C_0603_1608Metric_Pad1.08x0.95mm_HandSolder -> Capacitor_SMD:C_0402_1005Metric_Pad0.74x0.62mm_HandSolder; symbol bfr_capacitors:06035C104KAT2A -> bfr_capacitors:CL05B104KB54PNC; Created by capacitor_generator.py script using capacitor_bible_spec.txt -> capacitor_generator.py script using jlcbasic_additional_cap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; LCSC P/N C14663 -> C307331; Pretty Name 100nF 16V 0603 Capacitor -> 100nF X7R 50V 0402 Capacitor
- C1605: renamed from C1104; footprint Capacitor_SMD:C_0603_1608Metric_Pad1.08x0.95mm_HandSolder -> Capacitor_SMD:C_0402_1005Metric_Pad0.74x0.62mm_HandSolder; symbol bfr_capacitors:06035C104KAT2A -> bfr_capacitors:CL05B104KB54PNC; Created by capacitor_generator.py script using capacitor_bible_spec.txt -> capacitor_generator.py script using jlcbasic_additional_cap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; LCSC P/N C14663 -> C307331; Pretty Name 100nF 16V 0603 Capacitor -> 100nF X7R 50V 0402 Capacitor
Connections:
- net +3V3: now also C1601.1
- net GND: now also C1601.2
