File: power_protection.kicad_sch (KiCad schematic)
At the start: 10 parts, among them Q901 AO3401A, Q902 AO3401A

Commit message: fixed like a bunch of things, power and new xcvr and lights and other goodies, also started layout
Parts:
- removed D901: 4V7, Diode_SMD:D_SMB, symbol bfr_diodes:1SMB5917BT3G
- removed D902: 3V3, Diode_SMD:D_SMB, symbol bfr_diodes:1SMB5913BT3G
- removed D903, D904: BZT52C10-TP, Diode_SMD:D_SOD-123, symbol bfr_diodes:BZT52C10
- removed F901, F902: 500mA, Fuse:Fuse_1812_4532Metric, symbol bfr_utilities:0ZCG0050AF2C
- removed Q901, Q902: AO3401A, Package_TO_SOT_SMD:SOT-23-3, symbol Device:Q_PMOS_GSD
- removed R901, R902: 100k, Resistor_SMD:R_0603_1608Metric_Pad0.98x0.95mm_HandSolder, symbol bfr_resistors:RMCF0603FT100K
- added D1401, D1402: 20V, Diode_SMD:D_SMB, symbol bfr_diodes:1SMB5932BT3G
- added R1401: 470, Resistor_SMD:R_0402_1005Metric_Pad0.72x0.64mm_HandSolder, symbol bfr_resistors:RMCF0402FT470R
- added R1402, R1405: 360, Resistor_SMD:R_0603_1608Metric_Pad0.98x0.95mm_HandSolder, symbol bfr_resistors:RMCF0603FT360R
- added R1403, R1406: 390, Resistor_SMD:R_0603_1608Metric_Pad0.98x0.95mm_HandSolder, symbol bfr_resistors:RMCF0603FT390R
- added R1404: 270, Resistor_SMD:R_0603_1608Metric_Pad0.98x0.95mm_HandSolder, symbol bfr_resistors:RMCF0603FT270R
- added R1407, R1408: 100k, Resistor_SMD:R_0402_1005Metric_Pad0.72x0.64mm_HandSolder, symbol bfr_resistors:RMCF0402FT100K
- added U1401, U1402: TPS25961, Package_SON:WSON-6-1EP_2x2mm_P0.65mm_EP1x1.6mm, symbol bfr_power_ics:TPS25961
Connections:
- net 3V3_PROT: now also U1402.1 (VOUT)
- net 3V3_RAW: now also D1401.1 (K), R1404.2, U1402.6 (VIN)
- net 5V_PROT: now also U1401.1 (VOUT)
- net 5V_RAW: now also D1402.1 (K), R1401.2, U1401.6 (VIN)
- net GNDPWR: now also D1401.2 (A), D1402.2 (A), R1403.1, R1406.1, R1407.1, R1408.1, U1401.4 (GND), U1401.7 (EP), U1402.4 (GND), U1402.7 (EP)
- new net: R1401.1, R1402.2, U1401.5 (EN/UVLO)
- new net: R1405.1, R1406.2, U1402.2 (OVLO)
- new net: R1408.2, U1402.3 (ILIM)
- new net: R1404.1, R1405.2, U1402.5 (EN/UVLO)
- new net: R1402.1, R1403.2, U1401.2 (OVLO)
- new net: R1407.2, U1401.3 (ILIM)

Commit message: quicksave on some R.S. T.S. (mostly layout changes, small pin changes for better routing)
Connections:
- net GNDPWR: no longer D1401.2 (A), R1406.1, R1408.1, U1402.4 (GND), U1402.7 (EP)
- net 3V3_PROT renamed 3V3A_PROT
- net 3V3_RAW renamed 3V3A_RAW
- new net GND: D1401.2 (A), R1406.1, R1408.1, U1402.4 (GND), U1402.7 (EP)
Changed lines of the file:
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@@
 		)
 	)
-	(hierarchical_label "3V3_PROT"
+	(hierarchical_label "3V3A_PROT"
 		(shape input)
 		(at 231.14 123.19 0)
@@
 		)
 	)
-	(hierarchical_label "3V3_RAW"
+	(hierarchical_label "3V3A_RAW"
 		(shape input)
 		(at 90.17 123.19 180)
@@
 	(symbol
 		(lib_id "power:GNDPWR")
-		(at 96.52 146.05 0)
-		(unit 1)
-		(exclude_from_sim no)
-		(in_bom yes)
-		(on_board yes)
-		(dnp no)
-		(fields_autoplaced yes)
-		(property "Reference" "#PWR01401"
-			(at 96.52 151.13 0)
-			(effects
-				(font
-					(size 1.27 1.27)
-				)
-				(hide yes)
-			)
-		)
-		(property "Value" "GNDPWR"
-			(at 96.393 149.86 0)
-			(effects
-				(font
-					(size 1.27 1.27)
-				)
-			)
-		)
-		(property "Footprint" ""
-			(at 96.52 147.32 0)
-			(effects
-				(font
-					(size 1.27 1.27)
-				)
-				(hide yes)
-			)
-		)
-		(property "Datasheet" ""
-			(at 96.52 147.32 0)
-			(effects
-				(font
-					(size 1.27 1.27)
-				)
-				(hide yes)
-			)
-		)
-		(property "Description" "Power symbol creates a global label with name \"GNDPWR\" , global ground"
-			(at 96.52 146.05 0)
-			(effects
-				(font
-					(size 1.27 1.27)
-				)
-				(hide yes)
-			)
-		)
-		(pin "1"
-		)
-		(instances
-			(project "DU UC V1 - Minnow"
-				(path "/0aeff2df-21bc-4c76-95d6-83ff8577a8db/02d78338-99c8-4e1a-a94d-a7a2643a4fea/ef959e01-aa9b-4526-a9a5-a5bcea1528e7"
-					(reference "#PWR01401")
-					(unit 1)
-				)
-			)
-			(project "STM32F446 breakout V1 - Garibaldi"
-				(path "/6c37e641-6488-4ca1-9b36-326ba4e05a40/d78c720e-b278-4f28-a51f-ab95ac1d8264/ef959e01-aa9b-4526-a9a5-a5bcea1528e7"
-					(reference "#PWR050")
-					(unit 1)
-				)
-			)
-		)
-	)
-	(symbol
-		(lib_id "power:GNDPWR")
 		(at 97.79 106.68 0)
 		(unit 1)
@@
 					(unit 1)
 				)
+			)
+		)
+	)
+	(symbol
+		(lib_id "power:GND")
+		(at 96.52 146.05 0)
+		(unit 1)
+		(exclude_from_sim no)
+		(in_bom yes)
+		(on_board yes)
+		(dnp no)
+		(fields_autoplaced yes)
+		(property "Reference" "#PWR01803"
+			(at 96.52 152.4 0)
+			(effects
+				(font
+					(size 1.27 1.27)
+				)
+				(hide yes)
+			)
+		)
+		(property "Value" "GND"
+			(at 96.52 151.13 0)
+			(effects
+				(font
+					(size 1.27 1.27)
+				)
+			)
+		)
+		(property "Footprint" ""
+			(at 96.52 146.05 0)
+			(effects
+				(font
+					(size 1.27 1.27)
+				)
+				(hide yes)
+			)
+		)
+		(property "Datasheet" ""
+			(at 96.52 146.05 0)
+			(effects
+				(font
+					(size 1.27 1.27)
+				)
+				(hide yes)
+			)
+		)
+		(property "Description" "Power symbol creates a global label with name \"GND\" , ground"
+			(at 96.52 146.05 0)
+			(effects
+				(font
+					(size 1.27 1.27)
+				)
+				(hide yes)
+			)
+		)
+		(pin "1"
+		)
+		(instances
+			(project ""
+				(path "/0aeff2df-21bc-4c76-95d6-83ff8577a8db/02d78338-99c8-4e1a-a94d-a7a2643a4fea/ef959e01-aa9b-4526-a9a5-a5bcea1528e7"
+					(reference "#PWR01803")
+					(unit 1)
+				)

Commit message: laid out most of power, main xcvr, prob some other stuff
Connections:
- net GNDPWR is gone; now on net GND: D1402.2 (A), R1403.1, R1407.1, U1401.4 (GND), U1401.7 (EP)
Changed lines of the file:
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@@
+	)
+	(junction
+		(at 97.79 106.68)
+		(diameter 0)
+		(color 0 0 0 0)
 	)
 	(junction
@@
 	(junction
 		(at 130.81 146.05)
-		(diameter 0)
-		(color 0 0 0 0)
-	)
-	(junction
-		(at 97.79 106.68)
 		(diameter 0)
 		(color 0 0 0 0)
@@
 	)
 	(symbol
-		(lib_id "power:GNDPWR")
+		(lib_id "power:GND")
 		(at 97.79 106.68 0)
 		(unit 1)
@@
 		(dnp no)
 		(fields_autoplaced yes)
-		(property "Reference" "#PWR01402"
+		(property "Reference" "#PWR01804"
+			(at 97.79 113.03 0)
+			(effects
+				(font
+					(size 1.27 1.27)
+				)
+				(hide yes)
+			)
+		)
+		(property "Value" "GND"
 			(at 97.79 111.76 0)
 			(effects
@@
 					(size 1.27 1.27)
 				)
-				(hide yes)
-			)
-		)
-		(property "Value" "GNDPWR"
-			(at 97.663 110.49 0)
-			(effects
-				(font
-					(size 1.27 1.27)
-				)
 			)
 		)
 		(property "Footprint" ""
-			(at 97.79 107.95 0)
+			(at 97.79 106.68 0)
 			(effects
 				(font
@@
 		)
 		(property "Datasheet" ""
-			(at 97.79 107.95 0)
-			(effects
-				(font
-					(size 1.27 1.27)
-				)
-				(hide yes)
-			)
-		)
-		(property "Description" "Power symbol creates a global label with name \"GNDPWR\" , global ground"
+			(at 97.79 106.68 0)
+			(effects
+				(font
+					(size 1.27 1.27)
+				)
+				(hide yes)
+			)
+		)
+		(property "Description" "Power symbol creates a global label with name \"GND\" , ground"
 			(at 97.79 106.68 0)
 			(effects
@@
 			(project "DU UC V1 - Minnow"
 				(path "/0aeff2df-21bc-4c76-95d6-83ff8577a8db/02d78338-99c8-4e1a-a94d-a7a2643a4fea/ef959e01-aa9b-4526-a9a5-a5bcea1528e7"
-					(reference "#PWR01402")
+					(reference "#PWR01804")
 					(unit 1)
 				)
