File: DU UC V1 - Minnow.kicad_pcb (KiCad board)
At the start: 6 copper layers, 30 x 69.6 mm, 153 parts, among them J1701 MicroUSB, J1801 Conn_02x05_Odd_Even, J201 SODIMM-260, Q1301 BSS84, Q1501 BSS84, Q1502 BSS84, Q1701 MMBT3904, Q701 BSS84, Q702 BSS84, SW401 STLINK_RST, SW501 MCU_RST, U1101 74HC4051, U1401 TPS25961, U1402 TPS25961, U1501 TCAN334G, U1701 PSM712-LF-T7, U301 TPS7B8733QKVURQ1, U401 STM32F103CBTx, U501 STM32L552ZET6Q, U701 TCAN334G, U901 MX25R3235FM2xx1, Y401 8MHz 5pF, Y501 32.768kHz, 1.2pF, Y502 16MHz, 7pF

Commit message: i dont know what changed. dont ask me.
Parts:
- removed JP1201: LEDARR_EN, Jumper:SolderJumper-3_P1.3mm_Bridged2Bar12_Pad1.0x1.5mm_NumberLabels
- removed JP1202: LEDARR_A0, Jumper:SolderJumper-3_P1.3mm_Bridged2Bar12_Pad1.0x1.5mm_NumberLabels
- removed JP1203: LEDARR_A1, Jumper:SolderJumper-3_P1.3mm_Bridged2Bar12_Pad1.0x1.5mm_NumberLabels
- removed JP1204: LEDARR_A2, Jumper:SolderJumper-3_P1.3mm_Bridged2Bar12_Pad1.0x1.5mm_NumberLabels
- C504, JP501, R501: moved to F.Cu
- moved JP501 56.4 mm to (83.5, 129.8)
- moved JP502 44.3 mm to (92.9, 112.9), turned to -90 degrees
- moved JP503 41.1 mm to (101.6, 130.2)
- moved C306 7.37 mm to (116.6, 73.5), turned to -90 degrees
- moved C305 6.97 mm to (115.5, 73.5), turned to -90 degrees
- moved C304 6.95 mm to (114.3, 73.5), turned to -90 degrees
- moved R501 6.59 mm to (116.1, 114.1), turned to 0 degrees
- moved C302 3.78 mm to (114.3, 75.8), turned to 90 degrees
- moved C503 3.56 mm to (92.9, 109.3)
- moved C505 3.56 mm to (92.9, 108.2)
- moved R403 3.45 mm to (119.3, 80.6), turned to 180 degrees
- moved C502 2.56 mm to (103.7, 103.6)
- moved C501 2.56 mm to (105.3, 103.6)
- moved Y501 2.56 mm to (104.5, 106.5)
- moved C303 2.23 mm to (115.5, 75.8), turned to 90 degrees
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Connections:
- J201 pad 103: /SODIMM Connector/PC1 -> /SODIMM Connector/PC0
- J201 pad 107: /SODIMM Connector/PC2 -> /SODIMM Connector/PC1
- J201 pad 110: /SODIMM Connector/PC13 -> /SODIMM Connector/PC12
- J201 pad 111: /SODIMM Connector/PC3 -> /SODIMM Connector/PC2
- J201 pad 114: /SODIMM Connector/PC12 -> /SODIMM Connector/PC11
- J201 pad 115: /SODIMM Connector/PF12 -> /SODIMM Connector/PC3
- J201 pad 118: /SODIMM Connector/PC11 -> /SODIMM Connector/PC10
- J201 pad 119: /SODIMM Connector/PF13 -> /SODIMM Connector/PA0
- J201 pad 122: /SODIMM Connector/PC10 -> /SODIMM Connector/PA15
- J201 pad 123: /SODIMM Connector/PF14 -> /SODIMM Connector/PA1
- J201 pad 126: /SODIMM Connector/PA15 -> /SODIMM Connector/PA10
- J201 pad 127: /SODIMM Connector/PF15 -> /SODIMM Connector/PA2
- J201 pad 130: /SODIMM Connector/PA10 -> /SODIMM Connector/PA9
- J201 pad 131: /SODIMM Connector/PA0 -> /SODIMM Connector/PA3
- J201 pad 134: /SODIMM Connector/PA9 -> /SODIMM Connector/PA8
- J201 pad 135: /SODIMM Connector/PA1 -> /SODIMM Connector/PA4
- J201 pad 138: /SODIMM Connector/PA8 -> /SODIMM Connector/PC9
- J201 pad 139: /SODIMM Connector/PA2 -> /SODIMM Connector/PA5
- J201 pad 142: /SODIMM Connector/PC9 -> /SODIMM Connector/PC8
- J201 pad 143: /SODIMM Connector/PA3 -> /SODIMM Connector/PA6
- J201 pad 146: /SODIMM Connector/PC8 -> /SODIMM Connector/PC7
- J201 pad 147: /SODIMM Connector/PA4 -> /SODIMM Connector/PA7
- J201 pad 150: /SODIMM Connector/PC7 -> /SODIMM Connector/PC6
- J201 pad 151: /SODIMM Connector/PA5 -> /SODIMM Connector/PB0
- J201 pad 154: /SODIMM Connector/PC6 -> /SODIMM Connector/PG6
- J201 pad 155: /SODIMM Connector/PA6 -> /SODIMM Connector/PB1
- J201 pad 158: /SODIMM Connector/PG6 -> /SODIMM Connector/PG5
- J201 pad 159: /SODIMM Connector/PA7 -> /SODIMM Connector/PB2
- J201 pad 162: /SODIMM Connector/PG5 -> /SODIMM Connector/PG4
- J201 pad 163: /SODIMM Connector/PB0 -> /SODIMM Connector/PF11
- J201 pad 166: /SODIMM Connector/PG4 -> /SODIMM Connector/PG3
- J201 pad 167: /SODIMM Connector/PB1 -> /SODIMM Connector/PG0
- J201 pad 170: /SODIMM Connector/PG3 -> /SODIMM Connector/PG2
- J201 pad 171: /SODIMM Connector/PB2 -> /SODIMM Connector/PG1
- J201 pad 174: /SODIMM Connector/PG2 -> /SODIMM Connector/PD15
- J201 pad 175: /SODIMM Connector/PF11 -> /SODIMM Connector/PE7
- J201 pad 178: /SODIMM Connector/PD15 -> /SODIMM Connector/PD14
- J201 pad 179: /SODIMM Connector/PG0 -> /SODIMM Connector/PE8
- J201 pad 182: /SODIMM Connector/PD14 -> /SODIMM Connector/PD13
- J201 pad 183: /SODIMM Connector/PG1 -> /SODIMM Connector/PE9
- J201 pad 186: /SODIMM Connector/PD13 -> /SODIMM Connector/PD12
- J201 pad 187: /SODIMM Connector/PE7 -> /SODIMM Connector/PE10
- J201 pad 190: /SODIMM Connector/PD12 -> /SODIMM Connector/PD11
- J201 pad 191: /SODIMM Connector/PE8 -> /SODIMM Connector/PE11
- J201 pad 194: /SODIMM Connector/PD11 -> /SODIMM Connector/PD10
- J201 pad 195: /SODIMM Connector/PE9 -> /SODIMM Connector/PE12
- J201 pad 198: /SODIMM Connector/PD10 -> /SODIMM Connector/PD9
- J201 pad 199: /SODIMM Connector/PE10 -> /SODIMM Connector/PE13
- J201 pad 202: /SODIMM Connector/PD9 -> /SODIMM Connector/PD8
- J201 pad 203: /SODIMM Connector/PE11 -> /SODIMM Connector/PE14
- J201 pad 206: /SODIMM Connector/PD8 -> /SODIMM Connector/PB11
- J201 pad 207: /SODIMM Connector/PE12 -> /SODIMM Connector/PE15
- J201 pad 210: GND -> /SODIMM Connector/PB15
- J201 pad 211: /SODIMM Connector/PE13 -> /SODIMM Connector/PB10
- J201 pad 214: GND -> /SODIMM Connector/PB14
- J201 pad 215: /SODIMM Connector/PE14 -> GND
- J201 pad 218: GND -> /SODIMM Connector/PB13
- J201 pad 219: /SODIMM Connector/PE15 -> GND
- J201 pad 220: /SODIMM Connector/VBATT -> GND
- J201 pad 222: /SODIMM Connector/VBATT -> GND
- J201 pad 223: /SODIMM Connector/PB10 -> GND
- J201 pad 227: /SODIMM Connector/PB11 -> GND
- J201 pad 228: /SODIMM Connector/VDDIO -> GND
- J201 pad 231: /SODIMM Connector/PB13 -> GND
- J201 pad 235: /SODIMM Connector/PB14 -> GND
- J201 pad 236: GND -> /SODIMM Connector/VDDIO
- J201 pad 237: GND -> /SODIMM Connector/VDDUSB
- J201 pad 239: /SODIMM Connector/PB15 -> /SODIMM Connector/VDDUSB
- J201 pad 241: GND -> /SODIMM Connector/VDDUSB
- J201 pad 243: /SODIMM Connector/VDDUSB -> GND
- J201 pad 245: /SODIMM Connector/VDDUSB -> GND
- J201 pad 247: /SODIMM Connector/VDDUSB -> /SODIMM Connector/VBATT
- J201 pad 248: /SODIMM Connector/VREF -> GND
- J201 pad 249: GND -> /SODIMM Connector/VBATT
- J201 pad 55: /SODIMM Connector/PF0 -> /SODIMM Connector/PC13
- J201 pad 59: /SODIMM Connector/PF1 -> /SODIMM Connector/PF0
- J201 pad 63: /SODIMM Connector/PF2 -> /SODIMM Connector/PF1
- J201 pad 67: /SODIMM Connector/PF3 -> /SODIMM Connector/PF2
- J201 pad 71: /SODIMM Connector/PF4 -> /SODIMM Connector/PF3
- J201 pad 75: /SODIMM Connector/PF5 -> /SODIMM Connector/PF4
- J201 pad 79: /SODIMM Connector/PF6 -> /SODIMM Connector/PF5
- J201 pad 83: /SODIMM Connector/PF7 -> /SODIMM Connector/PF6
- J201 pad 87: /SODIMM Connector/PF8 -> /SODIMM Connector/PF7
- J201 pad 91: /SODIMM Connector/PF9 -> /SODIMM Connector/PF8
- J201 pad 95: /SODIMM Connector/PF10 -> /SODIMM Connector/PF9
- J201 pad 99: /SODIMM Connector/PC0 -> /SODIMM Connector/PF10
- U501 pad 47: /STM32L552ZET6Q/Peripherals/PF_IN12 -> /Debug LED Array/EN
- U501 pad 50: /STM32L552ZET6Q/Peripherals/PF_IN13 -> /Debug LED Array/A0
- U501 pad 51: /STM32L552ZET6Q/Peripherals/PF_IN14 -> /Debug LED Array/A1
- U501 pad 52: /STM32L552ZET6Q/Peripherals/PF_IN15 -> /Debug LED Array/A2
Routing:
- net /SODIMM Connector/PB9: track 0.00 -> 66.7 mm, vias 0 -> 1
- net /SODIMM Connector/PE0: track 0.00 -> 64.8 mm, vias 0 -> 2
- net /SODIMM Connector/PB8: track 0.00 -> 64.4 mm, vias 0 -> 1
- net /SODIMM Connector/PB7: track 0.00 -> 62.3 mm, vias 0 -> 1
- net /SODIMM Connector/PB6: track 0.00 -> 61.5 mm, vias 0 -> 1
- net /SODIMM Connector/PG13: track 0.00 -> 61.2 mm, vias 0 -> 1
- net /SODIMM Connector/PG14: track 0.00 -> 61.1 mm, vias 0 -> 1
- net /SODIMM Connector/PB5: track 0.00 -> 61.0 mm, vias 0 -> 1
- net /SODIMM Connector/PE1: track 0.00 -> 61.0 mm, vias 0 -> 2
- net /SODIMM Connector/PG12: track 0.00 -> 60.9 mm, vias 0 -> 1
- net /SODIMM Connector/PG15: track 0.00 -> 60.9 mm, vias 0 -> 1
- net /SODIMM Connector/PB4: track 0.00 -> 60.2 mm, vias 0 -> 1
- net /SODIMM Connector/PD7: track 0.00 -> 59.8 mm, vias 0 -> 1
- net /SODIMM Connector/PG9: track 0.00 -> 59.3 mm, vias 0 -> 1
- net /SODIMM Connector/PD6: track 0.00 -> 59.2 mm, vias 0 -> 1
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- added copper zone on B.Cu, net /5V_RAW
- added copper zone on In2.Cu, net /5V_RAW
Other:
- board text added: "PGOOD"
