File: sodimm.kicad_sch (KiCad schematic)
At the start: 3 parts, among them J201 SODIMM-260

Commit message: fucking shit bro i like expanded the board by 1mm and it still has no room fuck this bitchass crystal
Connections:
- net HOLD is gone; now on net GND: J201.216
- net WRITE_PROT is gone; now on net GND: J201.212
Changed lines of the file:
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@@
 	(wire
 		(pts
-			(xy 323.85 165.1) (xy 334.01 165.1)
-		)
-		(stroke
-			(width 0)
-			(type default)
-		)
-	)
-	(wire
-		(pts
 			(xy 288.29 205.74) (xy 288.29 203.2)
 		)
@@
 		)
 	)
-	(wire
-		(pts
-			(xy 323.85 160.02) (xy 334.01 160.02)
-		)
-		(stroke
-			(width 0)
-			(type default)
-		)
-	)
 	(bus
 		(pts
@@
 		)
 	)
-	(hierarchical_label "HOLD"
-		(shape input)
-		(at 334.01 165.1 0)
-		(effects
-			(font
-				(size 1.27 1.27)
-			)
-			(justify left)
-		)
-	)
 	(hierarchical_label "PF"
 		(shape bidirectional)
@@
 		)
 	)
-	(hierarchical_label "WRITE_PROT"
-		(shape input)
-		(at 334.01 160.02 0)
-		(effects
-			(font
-				(size 1.27 1.27)
-			)
-			(justify left)
-		)
-	)
 	(hierarchical_label "PE"
 		(shape bidirectional)
@@
 	(symbol
 		(lib_id "power:GND")
+		(at 323.85 160.02 90)
+		(unit 1)
+		(exclude_from_sim no)
+		(in_bom yes)
+		(on_board yes)
+		(dnp no)
+		(fields_autoplaced yes)
+		(property "Reference" "#PWR0327"
+			(at 330.2 160.02 0)
+			(effects
+				(font
+					(size 1.27 1.27)
+				)
+				(hide yes)
+			)
+		)
+		(property "Value" "GND"
+			(at 327.66 160.0199 90)
+			(effects
+				(font
+					(size 1.27 1.27)
+				)
+				(justify right)
+			)
+		)
+		(property "Footprint" ""
+			(at 323.85 160.02 0)
+			(effects
+				(font
+					(size 1.27 1.27)
+				)
+				(hide yes)
+			)
+		)
+		(property "Datasheet" ""
+			(at 323.85 160.02 0)
+			(effects
+				(font
+					(size 1.27 1.27)
+				)
+				(hide yes)
+			)
+		)
+		(property "Description" "Power symbol creates a global label with name \"GND\" , ground"
+			(at 323.85 160.02 0)
+			(effects
+				(font
+					(size 1.27 1.27)
+				)
+				(hide yes)
+			)
+		)
+		(pin "1"
+		)
+		(instances
+			(project "DU UC V1 - Minnow"
+				(path "/0aeff2df-21bc-4c76-95d6-83ff8577a8db/d936cc52-813e-4316-9119-269cdeafd53b"
+					(reference "#PWR0327")
+					(unit 1)
+				)
+			)
+		)
+	)
+	(symbol
+		(lib_id "power:GND")
 		(at 147.32 227.33 90)
 		(unit 1)
@@
 					(unit 1)
 				)
+			)
+		)
+	)
+	(symbol
+		(lib_id "power:GND")
+		(at 323.85 165.1 90)
+		(unit 1)
+		(exclude_from_sim no)
+		(in_bom yes)
+		(on_board yes)
+		(dnp no)
+		(fields_autoplaced yes)
+		(property "Reference" "#PWR0328"
+			(at 330.2 165.1 0)
+			(effects
+				(font
+					(size 1.27 1.27)
+				)
+				(hide yes)
+			)
+		)
+		(property "Value" "GND"
+			(at 327.66 165.0999 90)
+			(effects
+				(font
+					(size 1.27 1.27)
+				)
+				(justify right)
+			)
+		)
+		(property "Footprint" ""
+			(at 323.85 165.1 0)
+			(effects
+				(font
+					(size 1.27 1.27)
+				)
+				(hide yes)
+			)
+		)
+		(property "Datasheet" ""
+			(at 323.85 165.1 0)
+			(effects
+				(font
+					(size 1.27 1.27)
+				)
+				(hide yes)
+			)
+		)
+		(property "Description" "Power symbol creates a global label with name \"GND\" , ground"
+			(at 323.85 165.1 0)
+			(effects
+				(font
+					(size 1.27 1.27)
+				)
+				(hide yes)
+			)
+		)
+		(pin "1"
+		)
+		(instances
+			(project "DU UC V1 - Minnow"
+				(path "/0aeff2df-21bc-4c76-95d6-83ff8577a8db/d936cc52-813e-4316-9119-269cdeafd53b"
+					(reference "#PWR0328")
+					(unit 1)
+				)

Commit message: i dont know what changed. dont ask me.
Connections:
- net PF12 is gone; now on net PC3: J201.115
- net PF13 is gone; now on net PA0: J201.119
- net PF14 is gone; now on net PA1: J201.123
- net PF15 is gone; now on net PA2: J201.127
- net GND: now also J201.215, J201.219, J201.220, J201.222, J201.223, J201.227, J201.228, J201.231, J201.235, J201.243, J201.245, J201.248; no longer J201.210, J201.214, J201.218, J201.236, J201.237, J201.241, J201.249
- net PA0: no longer J201.131
- net PA1: no longer J201.135
- net PA10: now also J201.126; no longer J201.130
- net PA15: now also J201.122; no longer J201.126
- net PA2: no longer J201.139
- net PA3: now also J201.131; no longer J201.143
- net PA4: now also J201.135; no longer J201.147
- net PA5: now also J201.139; no longer J201.151
- net PA6: now also J201.143; no longer J201.155
- net PA7: now also J201.147; no longer J201.159
- net PA8: now also J201.134; no longer J201.138
- net PA9: now also J201.130; no longer J201.134
- net PB0: now also J201.151; no longer J201.163
- net PB1: now also J201.155; no longer J201.167
- net PB10: now also J201.211; no longer J201.223
- net PB11: now also J201.206; no longer J201.227
- net PB13: now also J201.218; no longer J201.231
- net PB14: now also J201.214; no longer J201.235
- net PB15: now also J201.210; no longer J201.239
- net PB2: now also J201.159; no longer J201.171
- net PC0: now also J201.103; no longer J201.99
- net PC1: now also J201.107; no longer J201.103
- net PC10: now also J201.118; no longer J201.122
- net PC11: now also J201.114; no longer J201.118
- net PC12: now also J201.110; no longer J201.114
- net PC13: now also J201.55; no longer J201.110
- net PC2: now also J201.111; no longer J201.107
- net PC3: no longer J201.111
- net PC6: now also J201.150; no longer J201.154
- net PC7: now also J201.146; no longer J201.150
- net PC8: now also J201.142; no longer J201.146
- net PC9: now also J201.138; no longer J201.142
- net PD10: now also J201.194; no longer J201.198
- net PD11: now also J201.190; no longer J201.194
- net PD12: now also J201.186; no longer J201.190
- net PD13: now also J201.182; no longer J201.186
- net PD14: now also J201.178; no longer J201.182
- net PD15: now also J201.174; no longer J201.178
- net PD8: now also J201.202; no longer J201.206
- net PD9: now also J201.198; no longer J201.202
- net PE10: now also J201.187; no longer J201.199
- net PE11: now also J201.191; no longer J201.203
- net PE12: now also J201.195; no longer J201.207
- net PE13: now also J201.199; no longer J201.211
- net PE14: now also J201.203; no longer J201.215
- net PE15: now also J201.207; no longer J201.219
- net PE7: now also J201.175; no longer J201.187
- net PE8: now also J201.179; no longer J201.191
- net PE9: now also J201.183; no longer J201.195
- net PF0: now also J201.59; no longer J201.55
- net PF1: now also J201.63; no longer J201.59
- net PF10: now also J201.99; no longer J201.95
- net PF11: now also J201.163; no longer J201.175
- net PF2: now also J201.67; no longer J201.63
- net PF3: now also J201.71; no longer J201.67
- net PF4: now also J201.75; no longer J201.71
- net PF5: now also J201.79; no longer J201.75
- net PF6: now also J201.83; no longer J201.79
- net PF7: now also J201.87; no longer J201.83
- net PF8: now also J201.91; no longer J201.87
- net PF9: now also J201.95; no longer J201.91
- net PG0: now also J201.167; no longer J201.179
- net PG1: now also J201.171; no longer J201.183
- net PG2: now also J201.170; no longer J201.174
- net PG3: now also J201.166; no longer J201.170
- net PG4: now also J201.162; no longer J201.166
- net PG5: now also J201.158; no longer J201.162
- net PG6: now also J201.154; no longer J201.158
- net VBATT: now also J201.247, J201.249; no longer J201.220, J201.222
- net VDDIO: now also J201.236; no longer J201.228
- net VDDUSB: now also J201.237, J201.239, J201.241; no longer J201.243, J201.245, J201.247
- net VREF: no longer J201.248
