File: ledarray.kicad_sch (KiCad schematic)
At the start: 19 parts, among them U1101 74HC4051

Commit message: laid out most of power, main xcvr, prob some other stuff
Connections:
- net LED_ARR_EN renamed EN
Changed lines of the file:
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@@
-		)
-	)
-	(label "{A[0..2],LED_ARR_EN}"
-		(at 60.96 95.25 0)
-		(effects
-			(font
-				(size 1.27 1.27)
-			)
-			(justify left bottom)
 		)
 	)
@@
 		)
 	)
-	(label "LED_ARR_EN"
-		(at 88.9 95.25 0)
+	(label "{EN, A[0..2]}"
+		(at 63.5 95.25 0)
 		(effects
 			(font
@@
 		(effects
 			(font
+				(size 1.27 1.27)
+			)
+			(justify left bottom)
+		)
+	)
+	(label "EN"
+		(at 88.9 95.25 0)
+		(effects
+			(font

Commit message: small schematic changes, need to reroute
Changed lines of the file:
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@@
-		)
-	)
-	(label "A1"
-		(at 121.92 100.33 0)
-		(effects
-			(font
-				(size 1.27 1.27)
-			)
-			(justify left bottom)
 		)
 	)
